File: directional-coupler/directional-coupler.sch (KiCad schematic (older format))
At the start: 71 parts

Commit message: Added and cleaned up DC schematic.
Parts:
- removed C? (x10): 100nF, Capacitor_SMD:C_0603_1608Metric_Pad1.05x0.95mm_HandSolder, symbol swr-meter-rescue:C_Small
- removed C?: 50pF, Capacitor_SMD:C_0603_1608Metric_Pad1.05x0.95mm_HandSolder, symbol swr-meter-rescue:C_Small
- removed C? (x2): 10nF, Capacitor_SMD:C_0603_1608Metric_Pad1.05x0.95mm_HandSolder, symbol swr-meter-rescue:C_Small
- removed C? (x8): 1nF, Capacitor_SMD:C_0603_1608Metric_Pad1.05x0.95mm_HandSolder, symbol swr-meter-rescue:C_Small
- removed C? (x2): 100pF, Capacitor_SMD:C_0603_1608Metric_Pad1.05x0.95mm_HandSolder, symbol swr-meter-rescue:C_Small
- removed D? (x2): 1N5711, Diode_SMD:D_SMA, symbol swr-meter-rescue:D_Schottky_Small_ALT
- removed J?: CONN_01X10, Connector_PinSocket_2.54mm:PinSocket_1x10_P2.54mm_Vertical, symbol swr-meter-rescue:CONN_01X10
- removed R?: 510Ω, Resistor_SMD:R_0603_1608Metric_Pad1.05x0.95mm_HandSolder, symbol swr-meter-rescue:R_Small
- removed R?: 49.9Ω, Resistor_SMD:R_0603_1608Metric_Pad1.05x0.95mm_HandSolder, symbol swr-meter-rescue:R_Small
- removed R?: 470Ω, Resistor_SMD:R_0603_1608Metric_Pad1.05x0.95mm_HandSolder, symbol swr-meter-rescue:R_Small
- removed R?: 100Ω, Resistor_SMD:R_0603_1608Metric_Pad1.05x0.95mm_HandSolder, symbol swr-meter-rescue:R_Small
- removed R?: 22Ω, Resistor_SMD:R_0603_1608Metric_Pad1.05x0.95mm_HandSolder, symbol swr-meter-rescue:R_Small
- removed R?: 33Ω, Resistor_SMD:R_0603_1608Metric_Pad1.05x0.95mm_HandSolder, symbol swr-meter-rescue:R_Small
- removed R? (x2): 1KΩ, Resistor_SMD:R_0603_1608Metric_Pad1.05x0.95mm_HandSolder, symbol swr-meter-rescue:R_Small
- removed R? (x2): 51Ω, Resistor_SMD:R_0603_1608Metric_Pad1.05x0.95mm_HandSolder, symbol swr-meter-rescue:R_Small
- removed R? (x2): 100KΩ, Resistor_SMD:R_0603_1608Metric_Pad1.05x0.95mm_HandSolder, symbol swr-meter-rescue:R_Variable
- removed R? (x4): 52.3Ω, Resistor_SMD:R_0603_1608Metric_Pad1.05x0.95mm_HandSolder, symbol swr-meter-rescue:R_Small
- removed R? (x2): 0Ω, Resistor_SMD:R_0603_1608Metric_Pad1.05x0.95mm_HandSolder, symbol swr-meter-rescue:R_Small
- removed R? (x2): 16.9Ω, Resistor_SMD:R_1206_3216Metric_Pad1.42x1.75mm_HandSolder, symbol swr-meter-rescue:R_Small
- removed R? (x4): 16.5Ω, Resistor_SMD:R_1206_3216Metric_Pad1.42x1.75mm_HandSolder, symbol swr-meter-rescue:R_Small
- removed R? (x2): 115Ω, Resistor_SMD:R_1206_3216Metric_Pad1.42x1.75mm_HandSolder, symbol swr-meter-rescue:R_Small
- removed R? (x4): 52.3Ω, Resistor_SMD:R_1206_3216Metric_Pad1.42x1.75mm_HandSolder, symbol swr-meter-rescue:R_Small
- removed R? (x2): 16.9Ω, Resistor_SMD:R_0805_2012Metric_Pad1.15x1.40mm_HandSolder, symbol swr-meter-rescue:R_Small
- removed R? (x4): 16.5Ω, Resistor_SMD:R_0805_2012Metric_Pad1.15x1.40mm_HandSolder, symbol swr-meter-rescue:R_Small
- removed U?: OPA695, TO_SOT_Packages_SMD:SOT-23-6, symbol swr-meter-rescue:OPA695
- removed U? (x2): AD8302, Housings_SSOP:TSSOP-14_4.4x5mm_Pitch0.65mm, symbol swr-meter-rescue:AD8302
- J? (x4): symbol swr-meter-rescue:CONN_COAXIAL -> directional-coupler-rescue:CONN_COAXIAL-swr-meter-rescue
- T? (x2): symbol swr-meter-rescue:Transformer_1P_1S -> directional-coupler-rescue:Transformer_1P_1S-swr-meter-rescue
Connections:
- net labels removed: +5V, fwd, fwd_env, fwd_preshft, fwd_pwr, fwd_ref, fwd_shft, mag, phase, refl, refl_env, refl_pwr, refl_ref, refl_shft, shft_mag, shft_phase, shft_vref, vref
- wire segments 274 -> 18
- no-connect marks 4 -> 0
Other:
- note removed: "180 Phase &\nMagnitude Detectors"
- note removed: "8dB Attenuator"
- note removed: "Directional Coupler"
- note removed: "Envelope Detector"
- note removed: "Optional Bypass"
- note removed: "Phase Shifter"
- note removed: "Power\nSplitter"
